File: PSU/TIPC PSU/TIPC PSU.kicad_pcb (KiCad board)
At the start: 2 copper layers, 35 parts, among them Q1 TO-92L

Commit message: Oh
Parts:
- removed the Q1 at (144.4, 91.1)
- removed the Q1 at (135.2, 88.6)
- removed the Q1 at (128.4, 90.6)
- added L1: L, Inductor_THT:L_Radial_D6.0mm_P4.00mm, F.Cu at (252.1, 25.5)
- added L2: L, Inductor_THT:L_Radial_D6.0mm_P4.00mm, F.Cu at (252.1, 33.5)
- added L3: L, Inductor_THT:L_Radial_D6.0mm_P4.00mm, F.Cu at (252.1, 41.5)
- added L4: L, Inductor_THT:L_Radial_D6.0mm_P4.00mm, F.Cu at (87.1, 76.5)
- added Q1: NPN, Package_TO_SOT_THT:TO-92L, F.Cu at (128.8, 90.8)
- added Q2: PNP, Package_TO_SOT_THT:TO-92L, F.Cu at (119.0, 76.6)
- added Q3: PNP, Package_TO_SOT_THT:TO-92L, F.Cu at (144.3, 90.9)
- added Q4: NPN, Package_TO_SOT_THT:TO-92L, F.Cu at (135.1, 88.5)
- added Q5: PNP, Package_TO_SOT_THT:TO-92L, F.Cu at (136.6, 78.6)
- added Q6: NPN, Package_TO_SOT_THT:TO-92L, F.Cu at (142.5, 78.5)
- added Q8: PNP, Package_TO_SOT_THT:TO-92L, F.Cu at (81.4, 66.7)
- added R17: R, Forgotten Machines:Resistor-Cap-P10.16mm_Horizontal, F.Cu at (142.7, 30.9)
- added R18: R, Forgotten Machines:Resistor-Cap-P10.16mm_Horizontal, F.Cu at (145.8, 30.9)
- added R19: R, Forgotten Machines:Resistor-Cap-P10.16mm_Horizontal, F.Cu at (148.8, 30.9)
- added R20: R, Forgotten Machines:Resistor-Cap-P10.16mm_Horizontal, F.Cu at (151.9, 30.9)
- added R21: R, Forgotten Machines:Resistor-Cap-P10.16mm_Horizontal, F.Cu at (154.9, 30.9)
- added R22: R, Forgotten Machines:Resistor-Cap-P10.16mm_Horizontal, F.Cu at (158.0, 30.9)
- added R23: R, Forgotten Machines:Resistor-Cap-P10.16mm_Horizontal, F.Cu at (161.1, 30.9)
- added R24: R, Forgotten Machines:Resistor-Cap-P10.16mm_Horizontal, F.Cu at (164.1, 30.9)
- added R25: R, Forgotten Machines:Resistor-Cap-P10.16mm_Horizontal, F.Cu at (167.2, 30.9)
- added R26: R, Forgotten Machines:Resistor-Cap-P10.16mm_Horizontal, F.Cu at (93.5, 79.8)
- added R27: R, Forgotten Machines:Resistor-Cap-P10.16mm_Horizontal, F.Cu at (173.3, 30.9)
- added R28: R, Forgotten Machines:Resistor-Cap-P10.16mm_Horizontal, F.Cu at (176.4, 30.9)
- added R29: R, Forgotten Machines:Resistor-Cap-P10.16mm_Horizontal, F.Cu at (179.4, 30.9)
- added R30: R, Forgotten Machines:Resistor-Cap-P10.16mm_Horizontal, F.Cu at (182.5, 30.9)
- added R31: R, Forgotten Machines:Resistor-Cap-P10.16mm_Horizontal, F.Cu at (185.5, 30.9)
- added R32: R, Forgotten Machines:Resistor-Cap-P10.16mm_Horizontal, F.Cu at (188.6, 30.9)
- added R33: R, Forgotten Machines:Resistor-Cap-P10.16mm_Horizontal, F.Cu at (191.7, 30.9)
- added R34: R, Forgotten Machines:Resistor-Cap-P10.16mm_Horizontal, F.Cu at (194.7, 30.9)
- added R35: R, Forgotten Machines:Resistor-Cap-P10.16mm_Horizontal, F.Cu at (197.8, 30.9)
- added R36: R, Forgotten Machines:Resistor-Cap-P10.16mm_Horizontal, F.Cu at (60.2, 90.6)
- added R37: R, Forgotten Machines:Resistor-Cap-P10.16mm_Horizontal, F.Cu at (63.2, 90.6)
- added R38: R, Forgotten Machines:Resistor-Cap-P10.16mm_Horizontal, F.Cu at (207.0, 30.9)
- added R39: R, Forgotten Machines:Resistor-Cap-P10.16mm_Horizontal, F.Cu at (210.0, 30.9)
- added R40: R, Forgotten Machines:Resistor-Cap-P10.16mm_Horizontal, F.Cu at (69.3, 90.6)
- moved D8 146.9 mm to (104.3, 31.0), turned to 90 degrees
- moved R8 141.5 mm to (110.4, 82.2), turned to 90 degrees
- moved R1 139.5 mm to (112.8, 30.9), turned to 90 degrees
- moved R10 137.2 mm to (114.0, 81.3), turned to 90 degrees
- moved R2 137.0 mm to (115.9, 30.9), turned to 90 degrees
- moved R3 134.5 mm to (119.0, 30.9), turned to 90 degrees
- moved D7 133.2 mm to (121.8, 71.1), turned to -90 degrees
- moved R4 132.2 mm to (122.0, 30.9), turned to 90 degrees
- moved D6 131.0 mm to (125.2, 71.1), turned to -90 degrees
- moved R6 129.9 mm to (125.1, 30.9), turned to 90 degrees
- moved R9 125.7 mm to (131.2, 30.9), turned to 90 degrees
- moved R12 122.3 mm to (136.8, 30.8), turned to 90 degrees
- moved R13 122.2 mm to (128.8, 81.4), turned to 90 degrees
- moved R14 119.1 mm to (131.8, 81.4), turned to 90 degrees
- moved JP1 74.2 mm to (226.1, 24.1)
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