File: PSU/TIPC PSU/TIPC PSU.kicad_pcb (KiCad board)
At the start: 2 copper layers, 67 parts, among them Q1 NPN, Q2 PNP, Q3 PNP, Q4 NPN, Q5 PNP, Q6 NPN, Q8 PNP

Commit message: o
Parts:
- added D10: D, Diode_THT:D_A-405_P10.16mm_Horizontal, F.Cu at (17.4, 21.1)
- added D11: D, Diode_THT:D_A-405_P10.16mm_Horizontal, F.Cu at (17.4, 25.4)
- added D12: D, Diode_THT:D_A-405_P10.16mm_Horizontal, F.Cu at (17.4, 29.6)
- added D13: D, Diode_THT:D_A-405_P10.16mm_Horizontal, F.Cu at (17.4, 33.9)
- added D14: D, Diode_THT:D_A-405_P10.16mm_Horizontal, F.Cu at (75.9, 67.6)
- added D15: D, Diode_THT:D_A-405_P10.16mm_Horizontal, F.Cu at (17.4, 42.4)
- added D9: D, Diode_THT:D_A-405_P10.16mm_Horizontal, F.Cu at (17.4, 16.9)
- added R41: R, Forgotten Machines:Resistor-Cap-P10.16mm_Horizontal, F.Cu at (58.7, 77.9)
