File: PSU/TIPC PSU/TIPC PSU.kicad_sch (KiCad schematic)
At the start: 0 parts

Commit message: lots
Parts:
- added C10: C_Small_US, Forgotten Machines:Resistor-Cap-P10.16mm_Horizontal, symbol Device:C_Small_US
- added C9: C_Small_US, Capacitor_THT:C_Disc_D4.3mm_W1.9mm_P5.00mm, symbol Device:C_Small_US
- added D1, D2, D3, D4, D5, D6, D7, D8: D, Diode_THT:D_A-405_P10.16mm_Horizontal, symbol Device:D
- added JP1, JP2, JP3, JP4, JP5, JP6: Jumper_2_Bridged, Forgotten Machines:Wire Jumper 0.325in, symbol Jumper:Jumper_2_Bridged
- added R1, R10, R11, R12, R13, R14, R15, R16, R2, R3, R4, R5, R6, R7, R8, R9: R, Forgotten Machines:Resistor-Cap-P10.16mm_Horizontal, symbol Device:R

Commit message: Oh
Parts:
- added L1, L2, L3, L4: L, Inductor_THT:L_Radial_D6.0mm_P4.00mm, symbol Device:L
- added Q1, Q4, Q6: NPN, Package_TO_SOT_THT:TO-92L, symbol Simulation_SPICE:NPN
- added Q2, Q3, Q5, Q8: PNP, Package_TO_SOT_THT:TO-92L, symbol Simulation_SPICE:PNP
- added R17, R18, R19, R20, R21, R22, R23, R24, R25, R26, R27, R28, R29, R30, R31, R32, R33, R34, R35, R36, R37, R38, R39, R40: R, Forgotten Machines:Resistor-Cap-P10.16mm_Horizontal, symbol Device:R

Commit message: o
Parts:
- added D10, D11, D12, D13, D14, D15, D9: D, Diode_THT:D_A-405_P10.16mm_Horizontal, symbol Device:D
- added R41: R, Forgotten Machines:Resistor-Cap-P10.16mm_Horizontal, symbol Device:R
